Commit message: add imu&slam_tool

File: description/ros2_control/diffbot.ros2_control.xacro (robot description, xacro)
@@ -8,15 +8,10 @@
             <param name="left_wheel_name">left_wheel_joint</param>
             <param name="right_wheel_name">right_wheel_joint</param>
-            <param name="loop_rate">30</param>
             <param name="device">/dev/ttyS7</param>
+            <param name="imu_name">diff_imu_joint</param>
+            <param name="wheel_distance">0.34</param>
+            <param name="wheel_radius">0.075</param>
             <param name="baud_rate">115200</param>
             <param name="timeout_ms">1000</param>
-            <param name="wheel_distance">0.34</param>
-            <param name="wheel_radius">0.075</param>
-            <param name="enc_counts_per_rev">3436</param>
-            <param name="pid_p">20</param>
-            <param name="pid_d">12</param>
-            <param name="pid_i">0</param>
-            <param name="pid_o">50</param>
         </hardware>
       </xacro:unless>
@@ -25,4 +20,5 @@
           <plugin>mock_components/GenericSystem</plugin>
           <param name="calculate_dynamics">true</param>
+          <param name="mock_sensor_commands">true</param>
         </hardware>
       </xacro:if>
@@ -37,4 +33,16 @@
         <state_interface name="velocity"/>
       </joint>
+      <joint name="diff_imu_joint">
+        <state_interface name="angular_velocity.x"/>
+        <state_interface name="angular_velocity.y"/>
+        <state_interface name="angular_velocity.z"/>
+        <state_interface name="linear_acceleration.x"/>
+        <state_interface name="linear_acceleration.y"/>
+        <state_interface name="linear_acceleration.z"/>
+        <state_interface name="orientation.w"/>
+        <state_interface name="orientation.x"/>
+        <state_interface name="orientation.y"/>
+        <state_interface name="orientation.z"/>
+      </joint>
     </ros2_control>
   </xacro:macro>

File: description/urdf/diffbot.urdf.xacro (robot description, xacro)
@@ -11,4 +11,6 @@
   <xacro:diffbot prefix="$(arg prefix)" />
   <xacro:diffbot_ros2_control
-    name="DiffBot" prefix="$(arg prefix)" use_mock_hardware="$(arg use_mock_hardware)"/>
+  name="DiffBot"
+  prefix="$(arg prefix)"
+  use_mock_hardware="$(arg use_mock_hardware)"/>
 </robot>

File: description/urdf/diffbot_description.urdf.xacro (robot description, xacro)
@@ -160,5 +160,51 @@
           izz="${caster_wheel_mass * 0.4 * (caster_wheel_radius * caster_wheel_radius)}"/>
         </inertial>
-      </link>
+    </link>
+    <joint name="diff_imu_joint" type="fixed">
+      <parent link="${prefix}base_link"/>
+      <child link="${prefix}diff_imu"/>
+      <origin xyz="${-base_radius/2 + caster_wheel_radius} 0 ${z_offset}" rpy="0 0 0"/>
+    </joint>
+    <link name="${prefix}diff_imu">
+      <collision>
+        <origin xyz="0 0 0" rpy="0 0 0"/>
+        <geometry>
+          <sphere radius="${caster_wheel_radius}"/>
+        </geometry>
+      </collision>
+      <visual>
+        <origin xyz="0 0 0" rpy="0 0 0"/>
+        <geometry>
+          <sphere radius="${caster_wheel_radius}"/>
+        </geometry>
+        <material name="white"/>
+      </visual>
+      <inertial>
+        <origin xyz="0 0 0" rpy="0 0 0"/>
+        <mass value="${caster_wheel_mass}"/>
+        <inertia
+          ixx="${caster_wheel_mass * 0.4 * (caster_wheel_radius * caster_wheel_radius)}" ixy="0.0" ixz="0.0"
+          iyy="${caster_wheel_mass * 0.4 * (caster_wheel_radius * caster_wheel_radius)}" iyz="0.0"
+          izz="${caster_wheel_mass * 0.4 * (caster_wheel_radius * caster_wheel_radius)}"/>
+        </inertial>
+    </link>
+    <joint name="lidar_joint" type="fixed">
+      <parent link="${prefix}base_link"/>
+      <child link="${prefix}laser_link"/>
+      <origin xyz="${-base_radius/2 + caster_wheel_radius} 0 ${z_offset}" rpy="0 0 0"/>
+    </joint>
+    <link name="laser_link">
+      <visual>
+          <geometry>
+              <cylinder radius="0.05" length="0.04"/>
+          </geometry>
+          <material name="red"/>
+      </visual>
+      <collision>
+          <geometry>
+              <cylinder radius="0.05" length="0.04"/>
+          </geometry>
+      </collision>
+    </link>
   </xacro:macro>
 </robot>
